File: AVE-NvidiaTX1-ISight360.sch (KiCad schematic (older format))
At the start: 0 parts

Commit message: Supplied Components to Ultrasonic bank
Changed lines of the file:
@@
 F0 "Power" 67
 F1 "Power.sch" 67
+F2 "5V" O R 3450 1300 67
 $EndSheet
-Text HLabel 3450 1300 0    67   Output ~ 13
-5V
 $Sheet
 S 1800 2950 850  2700
@@
 Text HLabel 7650 2150 2    67   Input ~ 13
 SCL
-$Sheet
-S 7600 3900 1250 1350
-U 58CA7E2A
-F0 "UltrasonicSensorBank" 67
-F1 "UltrasonicSensorBank.sch" 67
-$EndSheet
-Text HLabel 7600 4050 2    67   Input ~ 13
-PinTrigger4
-Text HLabel 7600 4250 2    67   Input ~ 13
-PinTrigger5
-Text HLabel 7600 4450 2    67   Input ~ 13
-PinTrigger6
-Text HLabel 7600 4700 2    67   Input ~ 13
-Echo
 Text HLabel 8800 1400 0    67   Input ~ 13
-5V
-Text HLabel 8850 4050 0    67   Input ~ 13
 5V
 Wire Wire Line
@@
 	4100 750  9350 750
 Wire Wire Line
-	9350 750  9350 4050
+	9350 750  9350 1400
+Wire Wire Line
+	9350 1400 9350 4050
 Wire Wire Line
 	9350 1400 8800 1400
@@
 	9350 4050 8850 4050
 Connection ~ 9350 1400
-Text HLabel 7600 4900 2    67   Input ~ 13
-PinTrigger7
 Wire Wire Line
 	2650 4900 7600 4900
@@
 Text Label 6500 3100 1    67   ~ 13
 SCL
+$Sheet
+S 7600 3900 1250 1350
+U 58CA7E2A
+F0 "UltrasonicSensorBank" 67
+F1 "UltrasonicSensorBank.sch" 67
+F2 "Echo" O L 7600 4700 67
+F3 "TriggerPin4" I L 7600 4050 67
+F4 "TriggerPin5" I L 7600 4250 67
+F5 "TriggerPin6" I L 7600 4450 67
+F6 "TriggerPin7" I L 7600 4900 67
+F7 "5V" I R 8850 4050 67
+$EndSheet
 $EndSCHEMATC

Commit message: Rev 1 Schematics
Other:
- note added: "Top Level Design"
Changed lines of the file:
@@
 Sheet 1 5
 Title "iSight360"
-Date "2017-03-16"
+Date "2017-03-17"
 Rev "A"
 Comp "Advanced Visual Electronics"
@@
 $EndDescr
 $Sheet
-S 1300 1050 2150 800
+S 1300 2050 2150 800
 U 58CA7067
 F0 "Power" 67
 F1 "Power.sch" 67
-F2 "5V" O R 3450 1300 67
+F2 "5V" O R 3450 2300 67
 $EndSheet
 $Sheet
-S 1800 2950 850  2700
+S 1800 3950 850  2700
 U 58CA7E0D
 F0 "GPIO Breakout" 67
 F1 "J20-Header-Breakout.sch" 67
+F2 "GPIO38" B R 2650 4200 60
+F3 "GPIO37" B R 2650 4400 60
+F4 "GPIO187" B R 2650 4600 60
+F5 "GPIO36" B R 2650 4850 60
+F6 "GPIO63" B R 2650 5100 60
+F7 "GPIO186" B R 2650 5350 60
+F8 "GPIO219" B R 2650 5650 60
+F9 "SCL" B R 2650 6400 60
+F10 "SDA" B R 2650 6200 60
+F11 "GPIO184" B R 2650 5900 60
 $EndSheet
-Text HLabel 2650 3200 0    67   BiDi ~ 13
-GPIO57
-Text HLabel 2650 3400 0    67   BiDi ~ 13
-GPIO160
-Text HLabel 2650 3600 0    67   BiDi ~ 13
-GPIO161
-Text HLabel 2650 3850 0    67   BiDi ~ 13
-GPIO162
-Text HLabel 2650 4100 0    67   BiDi ~ 13
-GPIO163
-Text HLabel 2650 4350 0    67   BiDi ~ 13
-GPIO164
-Text HLabel 2650 4650 0    67   BiDi ~ 13
-GPIO165
-Text HLabel 2650 4900 0    67   BiDi ~ 13
-GPIO166
-Text HLabel 2650 5200 0    67   BiDi ~ 13
-SDA
-Text HLabel 2650 5400 0    67   BiDi ~ 13
-SCL
-Text Notes 2200 5450 1    67   ~ 13
+Text Notes 2200 6450 1    67   ~ 13
 I2C
-Text Notes 2000 4100 1    67   ~ 13
+Text Notes 2000 5100 1    67   ~ 13
 GPIO
 $Sheet
-S 7650 1250 1150 1050
+S 7650 2250 1150 1050
 U 58CA7E20
 F0 "HapticMotorBank" 67
 F1 "HapticMotorBank.sch" 67
+F2 "PinTrigger2" I L 7650 2600 60
+F3 "5V" I R 8800 2400 60
+F4 "SDA" I L 7650 3000 60
+F5 "SCL" I L 7650 3150 60
+F6 "PinTrigger3" I L 7650 2800 60
+F7 "PinTrigger1" I L 7650 2400 60
 $EndSheet
-Text HLabel 7650 1400 2    67   Input ~ 13
-PinTrigger1
-Text HLabel 7650 1600 2    67   Input ~ 13
-PinTrigger2
-Text HLabel 7650 1800 2    67   Input ~ 13
-PinTrigger3
-Text HLabel 7650 2000 2    67   Input ~ 13
+Wire Wire Line
+	2650 4200 5000 4200
+Wire Wire Line
+	5000 4200 5000 2400
+Wire Wire Line
+	5000 2400 7650 2400
+Wire Wire Line
+	2650 4400 5200 4400
+Wire Wire Line
+	5200 4400 5200 2600
+Wire Wire Line
+	5200 2600 7650 2600
+Wire Wire Line
+	2650 4600 5450 4600
+Wire Wire Line
+	5450 4600 5450 2800
+Wire Wire Line
+	5450 2800 7650 2800
+Wire Wire Line
+	2650 6200 6150 6200
+Wire Wire Line
+	6150 6200 6150 3000
+Wire Wire Line
+	6150 3000 7650 3000
+Wire Wire Line
+	2650 6400 6500 6400
+Wire Wire Line
+	6500 6400 6500 3150
+Wire Wire Line
+	6500 3150 7650 3150
+Wire Wire Line
+	2650 4850 7400 4850
+Wire Wire Line
+	7400 4850 7400 5050
+Wire Wire Line
+	7400 5050 7600 5050
+Wire Wire Line
+	2650 5100 7350 5100
+Wire Wire Line
+	7350 5100 7350 5250
+Wire Wire Line
+	7350 5250 7600 5250
+Wire Wire Line
+	2650 5350 7350 5350
+Wire Wire Line
+	7350 5350 7350 5450
+Wire Wire Line
+	7350 5450 7600 5450
+Wire Wire Line
+	2650 5650 7300 5650
+Wire Wire Line
+	7300 5650 7300 5700
+Wire Wire Line
+	7300 5700 7600 5700
+Wire Wire Line
+	3450 2300 4100 2300
+Wire Wire Line
+	4100 2300 4100 1750
+Wire Wire Line
+	4100 1750 9350 1750
+Wire Wire Line
+	9350 1750 9350 5050
+Wire Wire Line
+	9350 2400 8800 2400
+Wire Wire Line
+	9350 5050 8850 5050
+Connection ~ 9350 2400
+Wire Wire Line
+	2650 5900 7600 5900
+Text Label 3750 5650 2    67   ~ 13
+Sensor_Input_Val
+Text Label 3700 5900 2    67   ~ 13
+Sensor_Trigger
+Text Notes 4850 5150 2    118  ~ 0
+Sensor MUX Control
+Text Notes 4850 4450 2    118  ~ 0
+Sensor MUX Control
+Text Label 6150 4050 1    67   ~ 13
 SDA
-Text HLabel 7650 2150 2    67   Input ~ 13
-SCL
-Text HLabel 8800 1400 0    67   Input ~ 13
-5V
-Wire Wire Line
-	2650 3200 5000 3200
-Wire Wire Line
-	5000 3200 5000 1400
-Wire Wire Line
-	5000 1400 7650 1400
-Wire Wire Line
-	2650 3400 5200 3400
-Wire Wire Line
-	5200 3400 5200 1600
-Wire Wire Line
-	5200 1600 7650 1600
-Wire Wire Line
-	2650 3600 5450 3600
-Wire Wire Line
-	5450 3600 5450 1800
-Wire Wire Line
-	5450 1800 7650 1800
-Wire Wire Line
-	2650 5200 6150 5200
-Wire Wire Line
-	6150 5200 6150 2000
-Wire Wire Line
-	6150 2000 7650 2000
-Wire Wire Line
-	2650 5400 6500 5400
-Wire Wire Line
-	6500 5400 6500 2150
-Wire Wire Line
-	6500 2150 7650 2150
-Wire Wire Line
-	2650 3850 7400 3850
-Wire Wire Line
-	7400 3850 7400 4050
-Wire Wire Line
-	7400 4050 7600 4050
-Wire Wire Line
-	2650 4100 7350 4100
-Wire Wire Line
-	7350 4100 7350 4250
-Wire Wire Line
-	7350 4250 7600 4250
-Wire Wire Line
-	2650 4350 7350 4350
-Wire Wire Line
-	7350 4350 7350 4450
-Wire Wire Line
-	7350 4450 7600 4450
-Wire Wire Line
-	2650 4650 7300 4650
-Wire Wire Line
-	7300 4650 7300 4700
-Wire Wire Line
-	7300 4700 7600 4700
-Wire Wire Line
-	3450 1300 4100 1300
-Wire Wire Line
-	4100 1300 4100 750
-Wire Wire Line
-	4100 750  9350 750
-Wire Wire Line
-	9350 750  9350 1400
-Wire Wire Line
-	9350 1400 9350 4050
-Wire Wire Line
-	9350 1400 8800 1400
-Wire Wire Line
-	9350 4050 8850 4050
-Connection ~ 9350 1400
-Wire Wire Line
-	2650 4900 7600 4900
-Text Label 3750 4650 2    67   ~ 13
-Sensor_Input_Val
-Text Label 3700 4900 2    67   ~ 13
-Sensor_Trigger
-Text Notes 4850 4150 2    118  ~ 0
-Sensor MUX Control
-Text Notes 4850 3450 2    118  ~ 0
-Sensor MUX Control
-Text Label 6150 3050 1    67   ~ 13
-SDA
-Text Label 6500 3100 1    67   ~ 13
+Text Label 6500 4050 1    67   ~ 13
 SCL
 $Sheet
-S 7600 3900 1250 1350
+S 7600 4900 1250 1350
 U 58CA7E2A
 F0 "UltrasonicSensorBank" 67
 F1 "UltrasonicSensorBank.sch" 67
-F2 "Echo" O L 7600 4700 67
-F3 "TriggerPin4" I L 7600 4050 67
-F4 "TriggerPin5" I L 7600 4250 67
-F5 "TriggerPin6" I L 7600 4450 67
-F6 "TriggerPin7" I L 7600 4900 67
-F7 "5V" I R 8850 4050 67
+F2 "Echo" O L 7600 5700 67
+F3 "TriggerPin4" I L 7600 5050 67
+F4 "TriggerPin5" I L 7600 5250 67
+F5 "TriggerPin6" I L 7600 5450 67
+F6 "TriggerPin7" I L 7600 5900 67
+F7 "5V" I R 8850 5050 67
 $EndSheet
+Text Notes 4800 1100 0    118  ~ 24
+Top Level Design
 $EndSCHEMATC

Commit message: Rev .99999 w/ Layout
Changed lines of the file:
@@
 F10 "SDA" B R 2650 6200 60
 F11 "GPIO184" B R 2650 5900 60
+F12 "5V" O L 1800 4100 60
+F13 "3.3V" O L 1800 4350 60
 $EndSheet
 Text Notes 2200 6450 1    67   ~ 13
@@
 	3450 2300 4100 2300
 Wire Wire Line
-	4100 2300 4100 1750
+	4100 1750 4100 3400
 Wire Wire Line
 	4100 1750 9350 1750
@@
 Text Notes 4800 1100 0    118  ~ 24
 Top Level Design
+Wire Wire Line
+	1800 4100 1350 4100
+Wire Wire Line
+	1350 4100 1350 3400
+Wire Wire Line
+	1350 3400 4100 3400
+Connection ~ 4100 2300
 $EndSCHEMATC
