File: Power.sch (KiCad schematic (older format))
At the start: 21 parts

Commit message: Supplied Components to Ultrasonic bank
Connections:
- net labels added: 5V
Changed lines of the file:
@@
 L +5F #PWR?
 U 1 1 58CA7CF4
-P 3150 5900
-F 0 "#PWR?" H 3150 5750 50  0001 C CNN
-F 1 "+5F" H 3150 6040 50  0000 C CNN
-F 2 "" H 3150 5900 50  0000 C CNN
-F 3 "" H 3150 5900 50  0000 C CNN
-	1    3150 5900
+P 3000 6100
+F 0 "#PWR?" H 3000 5950 50  0001 C CNN
+F 1 "+5F" H 3000 6240 50  0000 C CNN
+F 2 "" H 3000 6100 50  0000 C CNN
+F 3 "" H 3000 6100 50  0000 C CNN
+	1    3000 6100
 	1    0    0    -1
 $EndComp
@@
 Wire Wire Line
 	2300 6500 2300 6600
+Text HLabel 3150 5900 1    49   Output ~ 0
+5V
 $EndSCHEMATC

Commit message: Rev .99999 w/ Layout
Parts:
- C201, C202, C203, C204, C205, C206, C207, C208, C209, C210, C211, C212: renamed from C?; footprint (none) -> Capacitors_SMD:C_1206_HandSoldering
- D201: renamed from D?; footprint (none) -> Diodes_SMD:D_1206
- L201: renamed from L?; footprint (none) -> Inductors:Inductor_1212
- P201: renamed from P?; footprint (none) -> Connectors:JACK_ALIM
- R201, R202, R203, R204, R205: renamed from R?; footprint (none) -> Resistors_SMD:R_1206_HandSoldering
- gave numbers to parts that had none: 1
Connections:
- net labels removed: EN
- wire segments 61 -> 60
Changed lines of the file:
@@
 $EndDescr
 $Comp
-L TPS54231DR U?
+L TPS54231DR U201
 U 1 1 58CA7BEC
 P 5900 3800
-F 0 "U?" H 6150 3650 71  0000 C CNN
+F 0 "U201" H 6150 3650 71  0000 C CNN
 F 1 "TPS54231DR" H 5850 4750 60  0000 C CNN
 F 2 "SMD_Packages:SOIC-8-N" H 4850 3500 60  0001 C CNN
@@
 $EndComp
 $Comp
-L CONN_01X05 P?
+L CONN_01X05 P201
 U 1 1 58CA7BF3
 P 2350 3250
-F 0 "P?" H 2350 3550 50  0000 C CNN
+F 0 "P201" H 2350 3550 50  0000 C CNN
 F 1 "CONN_01X05" V 2450 3250 50  0000 C CNN
-F 2 "" H 2350 3250 50  0000 C CNN
+F 2 "Connectors:JACK_ALIM" H 2350 3250 50  0001 C CNN
 F 3 "" H 2350 3250 50  0000 C CNN
 	1    2350 3250
@@
 	3350 3300 5100 3300
 $Comp
-L +BATT #PWR?
+L +BATT #PWR01
 U 1 1 58CA7BFD
 P 3350 2750
-F 0 "#PWR?" H 3350 2600 50  0001 C CNN
+F 0 "#PWR01" H 3350 2600 50  0001 C CNN
 F 1 "+BATT" H 3350 2890 50  0000 C CNN
 F 2 "" H 3350 2750 50  0000 C CNN
@@
 $EndComp
 $Comp
-L GND #PWR?
+L GND #PWR02
 U 1 1 58CA7C03
 P 2750 3850
-F 0 "#PWR?" H 2750 3600 50  0001 C CNN
+F 0 "#PWR02" H 2750 3600 50  0001 C CNN
 F 1 "GND" H 2750 3700 50  0000 C CNN
 F 2 "" H 2750 3850 50  0000 C CNN
@@
 Connection ~ 2750 3450
 $Comp
-L GND #PWR?
+L GND #PWR03
 U 1 1 58CA7C11
 P 6750 4350
-F 0 "#PWR?" H 6750 4100 50  0001 C CNN
+F 0 "#PWR03" H 6750 4100 50  0001 C CNN
 F 1 "GND" H 6750 4200 50  0000 C CNN
 F 2 "" H 6750 4350 50  0000 C CNN
@@
 	6750 3000 6750 4350
 $Comp
-L C_Small C?
+L C_Small C204
 U 1 1 58CA7C19
 P 3350 3500
-F 0 "C?" H 3360 3570 50  0000 L CNN
+F 0 "C204" H 3360 3570 50  0000 L CNN
 F 1 "4.7uF" H 3360 3420 50  0000 L CNN
-F 2 "" H 3350 3500 50  0000 C CNN
+F 2 "Capacitors_SMD:C_1206_HandSoldering" H 3350 3500 50  0001 C CNN
 F 3 "" H 3350 3500 50  0000 C CNN
 	1    3350 3500
@@
 $EndComp
 $Comp
-L C_Small C?
+L C_Small C205
 U 1 1 58CA7C20
 P 3800 3500
-F 0 "C?" H 3810 3570 50  0000 L CNN
+F 0 "C205" H 3810 3570 50  0000 L CNN
 F 1 "4.7uF" H 3810 3420 50  0000 L CNN
-F 2 "" H 3800 3500 50  0000 C CNN
+F 2 "Capacitors_SMD:C_1206_HandSoldering" H 3800 3500 50  0001 C CNN
 F 3 "" H 3800 3500 50  0000 C CNN
 	1    3800 3500
@@
 $EndComp
 $Comp
-L C_Small C?
+L C_Small C206
 U 1 1 58CA7C27
 P 4150 3500
-F 0 "C?" H 4160 3570 50  0000 L CNN
+F 0 "C206" H 4160 3570 50  0000 L CNN
 F 1 "4.7uF" H 4160 3420 50  0000 L CNN
-F 2 "" H 4150 3500 50  0000 C CNN
+F 2 "Capacitors_SMD:C_1206_HandSoldering" H 4150 3500 50  0001 C CNN
 F 3 "" H 4150 3500 50  0000 C CNN
 	1    4150 3500
@@
 $EndComp
 $Comp
-L R_Small R?
+L R_Small R201
 U 1 1 58CA7C2E
 P 4550 3550
-F 0 "R?" H 4580 3570 50  0000 L CNN
+F 0 "R201" H 4580 3570 50  0000 L CNN
 F 1 "332k" H 4580 3510 50  0000 L CNN
-F 2 "" H 4550 3550 50  0000 C CNN
+F 2 "Resistors_SMD:R_1206_HandSoldering" H 4550 3550 50  0001 C CNN
 F 3 "" H 4550 3550 50  0000 C CNN
 	1    4550 3550
@@
 $EndComp
 $Comp
-L R_Small R?
+L R_Small R202
 U 1 1 58CA7C35
 P 4550 4100
-F 0 "R?" H 4580 4120 50  0000 L CNN
+F 0 "R202" H 4580 4120 50  0000 L CNN
 F 1 "68.1k" H 4580 4060 50  0000 L CNN
-F 2 "" H 4550 4100 50  0000 C CNN
+F 2 "Resistors_SMD:R_1206_HandSoldering" H 4550 4100 50  0001 C CNN
 F 3 "" H 4550 4100 50  0000 C CNN
 	1    4550 4100
@@
 	3800 3600 3800 3850
 $Comp
-L GND #PWR?
+L GND #PWR04
 U 1 1 58CA7C43
 P 3800 3850
-F 0 "#PWR?" H 3800 3600 50  0001 C CNN
+F 0 "#PWR04" H 3800 3600 50  0001 C CNN
 F 1 "GND" H 3800 3700 50  0000 C CNN
 F 2 "" H 3800 3850 50  0000 C CNN
@@
 	4550 4200 4550 4300
 Wire Wire Line
-	4300 3800 4900 3800
+	4550 3800 4900 3800
 Wire Wire Line
 	4900 3800 4900 3500
@@
 	4900 3500 5100 3500
 Connection ~ 4550 3800
-Wire Wire Line
-	4300 3800 4300 4300
-Text GLabel 4300 4300 3    60   Input ~ 0
-EN
-$Comp
-L GND #PWR?
+$Comp
+L GND #PWR05
 U 1 1 58CA7C53
 P 4550 4300
-F 0 "#PWR?" H 4550 4050 50  0001 C CNN
+F 0 "#PWR05" H 4550 4050 50  0001 C CNN
 F 1 "GND" H 4550 4150 50  0000 C CNN
 F 2 "" H 4550 4300 50  0000 C CNN
@@
 $EndComp
 $Comp
-L C_Small C?
+L C_Small C207
 U 1 1 58CA7C59
 P 5100 4100
-F 0 "C?" H 5110 4170 50  0000 L CNN
+F 0 "C207" H 5110 4170 50  0000 L CNN
 F 1 ".015uF" H 5110 4020 50  0000 L CNN
-F 2 "" H 5100 4100 50  0000 C CNN
+F 2 "Capacitors_SMD:C_1206_HandSoldering" H 5100 4100 50  0001 C CNN
 F 3 "" H 5100 4100 50  0000 C CNN
 	1    5100 4100
@@
 	4150 3650 4150 3600
 $Comp
-L C_Small C?
+L C_Small C208
 U 1 1 58CA7C66
 P 5800 2550
-F 0 "C?" H 5810 2620 50  0000 L CNN
+F 0 "C208" H 5810 2620 50  0000 L CNN
 F 1 ".1uF" H 5810 2470 50  0000 L CNN
-F 2 "" H 5800 2550 50  0000 C CNN
+F 2 "Capacitors_SMD:C_1206_HandSoldering" H 5800 2550 50  0001 C CNN
 F 3 "" H 5800 2550 50  0000 C CNN
 	1    5800 2550
@@
 	6450 2550 6450 3100
 $Comp
-L D_Zener_Small_ALT D?
+L D_Zener_Small_ALT D201
 U 1 1 58CA7C71
 P 7300 2800
-F 0 "D?" H 7300 2890 50  0000 C CNN
+F 0 "D201" H 7300 2890 50  0000 C CNN
 F 1 "B240A" H 7300 2710 50  0000 C CNN
-F 2 "" V 7300 2800 50  0000 C CNN
+F 2 "Diodes_SMD:D_1206" V 7300 2800 50  0001 C CNN
 F 3 "" V 7300 2800 50  0000 C CNN
 	1    7300 2800
@@
 $EndComp
 $Comp
-L C_Small C?
+L C_Small C210
 U 1 1 58CA7C78
 P 7750 2800
-F 0 "C?" H 7760 2870 50  0000 L CNN
+F 0 "C210" H 7760 2870 50  0000 L CNN
 F 1 "47uF" H 7760 2720 50  0000 L CNN
-F 2 "" H 7750 2800 50  0000 C CNN
+F 2 "Capacitors_SMD:C_1206_HandSoldering" H 7750 2800 50  0001 C CNN
 F 3 "" H 7750 2800 50  0000 C CNN
 	1    7750 2800
@@
 $EndComp
 $Comp
-L C_Small C?
+L C_Small C212
 U 1 1 58CA7C7F
 P 8100 2800
-F 0 "C?" H 8110 2870 50  0000 L CNN
+F 0 "C212" H 8110 2870 50  0000 L CNN
 F 1 "47uF" H 8110 2720 50  0000 L CNN
-F 2 "" H 8100 2800 50  0000 C CNN
+F 2 "Capacitors_SMD:C_1206_HandSoldering" H 8100 2800 50  0001 C CNN
 F 3 "" H 8100 2800 50  0000 C CNN
 	1    8100 2800
@@
 $EndComp
 $Comp
-L R_Small R?
+L R_Small R204
 U 1 1 58CA7C86
 P 8450 2800
-F 0 "R?" H 8480 2820 50  0000 L CNN
+F 0 "R204" H 8480 2820 50  0000 L CNN
 F 1 "10.2k" H 8480 2760 50  0000 L CNN
-F 2 "" H 8450 2800 50  0000 C CNN
+F 2 "Resistors_SMD:R_1206_HandSoldering" H 8450 2800 50  0001 C CNN
 F 3 "" H 8450 2800 50  0000 C CNN
 	1    8450 2800
@@
 $EndComp
 $Comp
-L L_Core_Iron_Small L?
+L L_Core_Iron_Small L201
 U 1 1 58CA7C8D
 P 7500 2600
-F 0 "L?" V 7600 2650 50  0000 L CNN
+F 0 "L201" V 7600 2650 50  0000 L CNN
 F 1 "10uH" V 7700 2550 50  0000 L CNN
-F 2 "" H 7500 2600 50  0000 C CNN
+F 2 "Inductors:Inductor_1212" H 7500 2600 50  0001 C CNN
 F 3 "" H 7500 2600 50  0000 C CNN
 	1    7500 2600
@@
 Connection ~ 8100 2600
 $Comp
-L R_Small R?
+L R_Small R205
 U 1 1 58CA7C9C
 P 8450 3200
-F 0 "R?" H 8480 3220 50  0000 L CNN
+F 0 "R205" H 8480 3220 50  0000 L CNN
 F 1 "R_Small" H 8480 3160 50  0000 L CNN
-F 2 "" H 8450 3200 50  0000 C CNN
+F 2 "Resistors_SMD:R_1206_HandSoldering" H 8450 3200 50  0001 C CNN
 F 3 "" H 8450 3200 50  0000 C CNN
 	1    8450 3200
@@
 	6450 3950 8450 3950
 $Comp
-L R_Small R?
+L R_Small R203
 U 1 1 58CA7CAE
 P 7200 3600
-F 0 "R?" H 7230 3620 50  0000 L CNN
+F 0 "R203" H 7230 3620 50  0000 L CNN
 F 1 "29.4k" H 7230 3560 50  0000 L CNN
-F 2 "" H 7200 3600 50  0000 C CNN
+F 2 "Resistors_SMD:R_1206_HandSoldering" H 7200 3600 50  0001 C CNN
 F 3 "" H 7200 3600 50  0000 C CNN
 	1    7200 3600
@@
 $EndComp
 $Comp
-L C_Small C?
+L C_Small C209
 U 1 1 58CA7CB5
 P 7200 3300
-F 0 "C?" H 7210 3370 50  0000 L CNN
+F 0 "C209" H 7210 3370 50  0000 L CNN
 F 1 "1000pF" H 7210 3220 50  0000 L CNN
-F 2 "" H 7200 3300 50  0000 C CNN
+F 2 "Capacitors_SMD:C_1206_HandSoldering" H 7200 3300 50  0001 C CNN
 F 3 "" H 7200 3300 50  0000 C CNN
 	1    7200 3300
@@
 $EndComp
 $Comp
-L C_Small C?
+L C_Small C211
 U 1 1 58CA7CBC
 P 7750 3300
-F 0 "C?" H 7760 3370 50  0000 L CNN
+F 0 "C211" H 7760 3370 50  0000 L CNN
 F 1 "47pF" H 7760 3220 50  0000 L CNN
-F 2 "" H 7750 3300 50  0000 C CNN
+F 2 "Capacitors_SMD:C_1206_HandSoldering" H 7750 3300 50  0001 C CNN
 F 3 "" H 7750 3300 50  0000 C CNN
 	1    7750 3300
@@
 Switch mode power supply 19->5
 $Comp
-L +5V #PWR?
+L +5V #PWR06
 U 1 1 58CA7CD3
 P 9350 2600
-F 0 "#PWR?" H 9350 2450 50  0001 C CNN
+F 0 "#PWR06" H 9350 2450 50  0001 C CNN
 F 1 "+5V" H 9350 2740 50  0000 C CNN
 F 2 "" H 9350 2600 50  0000 C CNN
@@
 $EndComp
 $Comp
-L C_Small C?
+L C_Small C201
 U 1 1 58CA7CD9
 P 1850 6200
-F 0 "C?" H 1860 6270 50  0000 L CNN
+F 0 "C201" H 1860 6270 50  0000 L CNN
 F 1 "10uF" H 1860 6120 50  0000 L CNN
-F 2 "" H 1850 6200 50  0000 C CNN
+F 2 "Capacitors_SMD:C_1206_HandSoldering" H 1850 6200 50  0001 C CNN
 F 3 "" H 1850 6200 50  0000 C CNN
 	1    1850 6200
@@
 $EndComp
 $Comp
-L C_Small C?
+L C_Small C202
 U 1 1 58CA7CE0
 P 2300 6200
-F 0 "C?" H 2310 6270 50  0000 L CNN
+F 0 "C202" H 2310 6270 50  0000 L CNN
 F 1 "100uF" H 2310 6120 50  0000 L CNN
-F 2 "" H 2300 6200 50  0000 C CNN
+F 2 "Capacitors_SMD:C_1206_HandSoldering" H 2300 6200 50  0001 C CNN
 F 3 "" H 2300 6200 50  0000 C CNN
 	1    2300 6200
@@
 $EndComp
 $Comp
-L C_Small C?
+L C_Small C203
 U 1 1 58CA7CE7
 P 2700 6200
-F 0 "C?" H 2710 6270 50  0000 L CNN
+F 0 "C203" H 2710 6270 50  0000 L CNN
 F 1 ".1uF" H 2710 6120 50  0000 L CNN
-F 2 "" H 2700 6200 50  0000 C CNN
+F 2 "Capacitors_SMD:C_1206_HandSoldering" H 2700 6200 50  0001 C CNN
 F 3 "" H 2700 6200 50  0000 C CNN
 	1    2700 6200
@@
 $EndComp
 $Comp
-L +5V #PWR?
+L +5V #PWR07
 U 1 1 58CA7CEE
 P 1550 5950
-F 0 "#PWR?" H 1550 5800 50  0001 C CNN
+F 0 "#PWR07" H 1550 5800 50  0001 C CNN
 F 1 "+5V" H 1550 6090 50  0000 C CNN
 F 2 "" H 1550 5950 50  0000 C CNN
@@
 $EndComp
 $Comp
-L +5F #PWR?
+L +5F #PWR08
 U 1 1 58CA7CF4
 P 3000 6100
-F 0 "#PWR?" H 3000 5950 50  0001 C CNN
+F 0 "#PWR08" H 3000 5950 50  0001 C CNN
 F 1 "+5F" H 3000 6240 50  0000 C CNN
 F 2 "" H 3000 6100 50  0000 C CNN
@@
 Connection ~ 2300 6450
 $Comp
-L GND #PWR?
+L GND #PWR09
 U 1 1 58CA7D05
 P 2300 6600
-F 0 "#PWR?" H 2300 6350 50  0001 C CNN
+F 0 "#PWR09" H 2300 6350 50  0001 C CNN
 F 1 "GND" H 2300 6450 50  0000 C CNN
 F 2 "" H 2300 6600 50  0000 C CNN
@@
 Text HLabel 3150 5900 1    49   Output ~ 0
 5V
+Connection ~ 3350 3050
 $EndSCHEMATC
