File: AVE-NvidiaTX1-ISight360-Backup.kicad_pcb (KiCad board)
At the start: 2 copper layers, 71.1 x 106.7 mm, 22 parts, among them P201 CONN_02X20, P401 Ultrasonic 1, P402 Ultrasonic2, P403 Ultrasonic3, P404 Ultrasonic4, P405 Ultrasonic5, P406 Ultrasonic6, U301 CD4051B, U302 DRV2605L(breakout), U303 DRV2605L(breakout)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

Commit message: Layout Done
Minor Tweaks were made to Schematic
Routing:
- net GND: track 287.1 -> 267.5 mm, vias 16 -> 12
- removed copper zone on F.Cu, net GND
Changed lines of the file:
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@@
   (general
     (links 89)
-    (no_connects 1)
+    (no_connects 4)
     (area 110.414999 35.484999 181.685001 142.315001)
     (thickness 1.6)
     (drawings 4)
-    (tracks 502)
+    (tracks 491)
     (zones 0)
     (modules 22)
@@
   (segment (start 163.322 59.182) (end 161.798 59.182) (width 0.508) (layer F.Cu) (net 0))
   (segment (start 163.322 59.182) (end 165.1 60.96) (width 0.508) (layer F.Cu) (net 0))
-  (via (at 121.412 86.36) (size 0.6) (drill 0.4) (layers F.Cu B.Cu) (net 1))
-  (segment (start 129.54 86.36) (end 122.936 86.36) (width 0.635) (layer B.Cu) (net 1))
-  (segment (start 122.936 86.36) (end 121.412 86.36) (width 0.635) (layer B.Cu) (net 1))
-  (segment (start 157.48 107.95) (end 157.48 115.57) (width 0.508) (layer B.Cu) (net 1))
-  (via (at 156.972 116.078) (size 0.6) (drill 0.4) (layers F.Cu B.Cu) (net 1))
-  (segment (start 157.48 115.57) (end 156.972 116.078) (width 0.508) (layer B.Cu) (net 1))
-  (segment (start 154.94 134.62) (end 157.734 131.826) (width 0.508) (layer B.Cu) (net 1))
-  (via (at 155.702 127) (size 0.6) (drill 0.4) (layers F.Cu B.Cu) (net 1))
-  (segment (start 157.48 127) (end 155.702 127) (width 0.508) (layer F.Cu) (net 1))
-  (segment (start 158.496 128.016) (end 157.48 127) (width 0.508) (layer F.Cu) (net 1))
-  (segment (start 158.496 131.064) (end 158.496 128.016) (width 0.508) (layer F.Cu) (net 1))
-  (segment (start 157.734 131.826) (end 158.496 131.064) (width 0.508) (layer F.Cu) (net 1))
-  (via (at 157.734 131.826) (size 0.6) (drill 0.4) (layers F.Cu B.Cu) (net 1))
   (segment (start 166.624 87.122) (end 166.624 88.392) (width 0.508) (layer F.Cu) (net 1))
   (segment (start 171.196 86.36) (end 169.672 84.836) (width 0.508) (layer B.Cu) (net 1))
@@
   (segment (start 164.084 66.04) (end 165.1 66.04) (width 0.635) (layer B.Cu) (net 1))
   (segment (start 152.4 66.04) (end 164.084 66.04) (width 0.635) (layer B.Cu) (net 1))
+  (segment (start 122.936 86.36) (end 121.412 86.36) (width 0.635) (layer B.Cu) (net 1))
+  (segment (start 129.54 86.36) (end 122.936 86.36) (width 0.635) (layer B.Cu) (net 1))
   (segment (start 171.45 90.424) (end 171.704 90.424) (width 0.508) (layer B.Cu) (net 2))
   (segment (start 165.608 92.456) (end 167.64 90.424) (width 0.635) (layer B.Cu) (net 2))
@@
       )
     )
-  )
-  (zone (net 1) (net_name GND) (layer F.Cu) (hatch edge 0.508)
-    (connect_pads (clearance 0.508))
-    (min_thickness 0.254)
-    (fill yes (arc_segments 16) (thermal_gap 0.508) (thermal_bridge_width 0.508))
-    (polygon
-      (pts
-        (xy 178.816 141.224) (xy 113.03 141.224) (xy 111.252 139.7) (xy 111.252 37.592) (xy 112.268 36.322)
-        (xy 179.578 36.322) (xy 180.848 37.338) (xy 180.848 139.446) (xy 179.324 141.224)
-      )
-    )
