File: Kicad Schematics/UltrasonicSensorBank.sch (KiCad schematic (older format))
At the start: 11 parts, among them P501 Ultrasonic 1, P502 Ultrasonic2, P503 Ultrasonic3, P504 Ultrasonic4, P505 Ultrasonic5, P506 Ultrasonic6, U501 74LVC1T45, U502 74LS251

Commit message: Reduced number of components
Parts:
- removed JP501: Jumper_NC_Dual, Pin_Headers:Pin_Header_Straight_1x03_Pitch2.54mm_SMD_Pin1Left, symbol Jumper_NC_Dual
- removed U501: 74LVC1T45, TO_SOT_Packages_SMD:SOT-363_SC-70-6_Handsoldering, symbol 74LVC1T45
- removed U502: 74LS251, SMD_Packages:SO-16-N, symbol 74LS251
- added JP401: Usonic Power Select, Pin_Headers:Pin_Header_Straight_1x03_Pitch2.54mm, symbol Jumper_NC_Dual
- added R403: 100K, Resistors_SMD:R_1206_HandSoldering, symbol R_Small
- added R404: 10K, Resistors_SMD:R_1206_HandSoldering, symbol R_Small
- added U401: LM4250, SMD_Packages:SOIC-8-N, symbol LM741
- added U402: CD4051B, Housings_DIP:DIP-16_W7.62mm_LongPads, symbol CD4051B
- R402: renamed from R502; value 10K -> 20K
- renumbered P501 to P401, P502 to P402, P503 to P403, P504 to P404, P505 to P405, P506 to P406, R501 to R401
Connections:
- net labels added: 3.3V, U-Power, Ultrasonic_Trigger, Ultrasonic_Vin
- net labels removed: +1V2, +5F, Trigger
- wire segments 58 -> 74
- no-connect marks 3 -> 6
Other:
- note added: "3.3V"
- note added: "5V"
- note added: "5v -> 3.3v Divider"
- note added: "Comparator Circuit to Boost Voltage"
- note added: "Selectable Power Source"
- note added: "Selector Pins"
- note removed: "Bidirectional Level Shifter"
- note removed: "Set Vcc(a) "HIGH" for A->B Transmission"

Commit message: Rev C Update
Connections:
- net labels added: UltrasonicEcho1, UltrasonicEcho2, UltrasonicEcho3, UltrasonicEcho4, UltrasonicEcho5, UltrasonicEcho6
- wire segments 74 -> 81
Other:
- note added: "Ultrasonic Sensor Breakouts"
Changed lines of the file:
@@
 $Descr A4 11693 8268
 encoding utf-8
-Sheet 4 4
+Sheet 4 5
 Title "Ultrasonic Sensor Bank"
-Date "2017-03-17"
-Rev "A"
+Date "2000-12-31"
+Rev "C"
 Comp "Advanced Visual Electronics"
 Comment1 "Designer: Christian Aguilar"
@@
 	6400 3500 6400 6100
 Wire Notes Line
-	6400 6100 1300 6100
+	6400 6100 850  6100
 Wire Notes Line
 	1300 6100 1300 3500
@@
 $EndComp
 NoConn ~ 8300 1800
+Wire Wire Line
+	2500 6600 1300 6600
+Wire Wire Line
+	1300 6750 2500 6750
+Wire Wire Line
+	2500 6900 1300 6900
+Wire Wire Line
+	1300 7050 2500 7050
+Wire Wire Line
+	2500 7200 1300 7200
+Wire Wire Line
+	1300 7350 2500 7350
+Text Label 1750 6600 0    30   ~ 0
+Echo1
+Text Label 1750 6750 0    30   ~ 0
+Echo2
+Text Label 1750 6900 0    30   ~ 0
+Echo3
+Text Label 1750 7050 0    30   ~ 0
+Echo4
+Text Label 1750 7200 0    30   ~ 0
+Echo5
+Text Label 1750 7350 0    30   ~ 0
+Echo6
+Text HLabel 2500 6600 2    30   Output ~ 0
+UltrasonicEcho1
+Text HLabel 2500 6750 2    30   Output ~ 0
+UltrasonicEcho2
+Text HLabel 2500 6900 2    30   Output ~ 0
+UltrasonicEcho3
+Text HLabel 2500 7050 2    30   Output ~ 0
+UltrasonicEcho4
+Text HLabel 2500 7200 2    30   Output ~ 0
+UltrasonicEcho5
+Text HLabel 2500 7350 2    30   Output ~ 0
+UltrasonicEcho6
+Wire Notes Line
+	850  6100 850  7600
+Wire Notes Line
+	850  7600 4400 7600
+Wire Notes Line
+	4400 7600 4400 6100
+Text Notes 2800 6300 2    67   ~ 0
+Ultrasonic Sensor Breakouts
+Wire Wire Line
+	1300 7500 2450 7500
+Text Label 1750 7500 0    30   ~ 0
+Ultrasonic_Trigger
 $EndSCHEMATC
